Commit message: rtabmap

File: description/camera.xacro (robot description, xacro)
@@ -34,5 +34,5 @@
   <!-- Camera -->
   <joint name="camera_joint" type="fixed">
-    <parent link="base_link" />
+    <parent link="chassis_link" />
     <child link="camera_link" />
     <origin xyz="${wheel_offset_x} 0 ${wheel_offset_z}" rpy="0 0 0"/>
@@ -217,5 +217,5 @@
       <colorUpdateRate>60.0</colorUpdateRate>
       <infraredUpdateRate>60.0</infraredUpdateRate>
-      <depthTopicName>depth/image_rect_raw</depthTopicName>
+      <depthTopicName>aligned_depth_to_color/image_raw</depthTopicName>
       <depthCameraInfoTopicName>depth/camera_info</depthCameraInfoTopicName>
       <colorTopicName>color/image_raw</colorTopicName>
@@ -230,5 +230,5 @@
       <rangeMaxDepth>10.0</rangeMaxDepth>
       <pointCloud>true</pointCloud>
-      <pointCloudTopicName>depth/points</pointCloudTopicName>
+      <pointCloudTopicName>depth/color/points</pointCloudTopicName>
       <pointCloudCutoff>0.5</pointCloudCutoff>
     </plugin>

File: description/gazebo_control.xacro (robot description, xacro)
@@ -6,5 +6,5 @@
             <left_joint>left_wheel_joint</left_joint>
             <right_joint>right_wheel_joint</right_joint>
-            <wheel_separation>0.18</wheel_separation>
+            <wheel_separation>0.2</wheel_separation>
             <wheel_diameter>0.065</wheel_diameter>
             <!-- Limits -->

File: description/robot.urdf.xacro (robot description, xacro)
@@ -4,3 +4,5 @@
     <xacro:include filename="ros2_control.xacro" />
     <xacro:include filename="camera.xacro" />
+    <xacro:include filename="imu.xacro" />
+    <!-- <xacro:include filename="lidar.xacro" /> -->
 </robot>

File: description/robot_core.xacro (robot description, xacro)
@@ -14,5 +14,5 @@
     <xacro:property name="caster_wheel_radius" value="0.0125"/>
     <xacro:property name="caster_wheel_mass" value="0.01"/>
-    <xacro:property name="caster_wheel_offset_x" value="0.08"/>
+    <xacro:property name="caster_wheel_offset_x" value="0.05"/>
     <xacro:property name="caster_wheel_offset_z" value="${wheel_offset_z - wheel_radius + caster_wheel_radius}"/>
     <!-- BASE LINK -->

File: description/ros2_control.xacro (robot description, xacro)
@@ -1,25 +1,77 @@
 <?xml version="1.0"?>
 <robot xmlns:xacro="http://www.ros.org/wiki/xacro">
-    <ros2_control name="GazeboSystem" type="system">
+    <xacro:unless value="$(arg sim_mode)">
+        <ros2_control name="RealRobot" type="system">
+            <hardware>
+                <plugin>diffdrive_arduino/DiffDriveArduino</plugin>
+                <param name="left_wheel_name">left_wheel_joint</param>
+                <param name="right_wheel_name">right_wheel_joint</param>
+                <param name="loop_rate">30</param>
+                <param name="device">/dev/ttyUSB0</param>
+                <param name="baud_rate">57600</param>
+                <param name="timeout">1000</param>
+                <param name="enc_counts_per_rev">3436</param>
+            </hardware>
+            <joint name="left_wheel_joint">
+                <command_interface name="velocity">
+                    <param name="min">-10</param>
+                    <param name="max">10</param>
+                </command_interface>
+                <state_interface name="velocity"/>
+                <state_interface name="position"/>
+            </joint>
+            <joint name="right_wheel_joint">
+                <command_interface name="velocity">
+                    <param name="min">-10</param>
+                    <param name="max">10</param>
+                </command_interface>
+                <state_interface name="velocity"/>
+                <state_interface name="position"/>
+            </joint>
+        </ros2_control>
+        <!-- MPU6050 sensor-->
+        <ros2_control name='MPU6050' type='sensor'>
         <hardware>
-            <plugin>gazebo_ros2_control/GazeboSystem</plugin>
+            <plugin>lidarbot_bringup/MPU6050Hardware</plugin>
+            <param name='sensor_name'>mpu6050</param>
+            <param name='frame_id'>imu_link</param>
         </hardware>
-        <joint name="left_wheel_joint">
-            <command_interface name="velocity">
-                <param name="min">-10</param>
-                <param name="max">10</param>
-            </command_interface>
-            <state_interface name="velocity"/>
-            <state_interface name="position"/>
-        </joint>
-        <joint name="right_wheel_joint">
-            <command_interface name="velocity">
-                <param name="min">-10</param>
-                <param name="max">10</param>
-            </command_interface>
-            <state_interface name="velocity"/>
-            <state_interface name="position"/>
-        </joint>
-    </ros2_control>
+        <sensor name='mpu6050'>
+            <state_interface name='orientation.x'/>
+            <state_interface name='orientation.y'/>
+            <state_interface name='orientation.z'/>
+            <state_interface name='orientation.w'/>
+            <state_interface name='angular_velocity.x'/>
+            <state_interface name='angular_velocity.y'/>
+            <state_interface name='angular_velocity.z'/>
+            <state_interface name='linear_acceleration.x'/>
+            <state_interface name='linear_acceleration.y'/>
+            <state_interface name='linear_acceleration.z'/>
+        </sensor>
+        </ros2_control>
+    </xacro:unless>
+    <xacro:if value="$(arg sim_mode)">
+        <ros2_control name="GazeboSystem" type="system">
+            <hardware>
+                <plugin>gazebo_ros2_control/GazeboSystem</plugin>
+            </hardware>
+            <joint name="left_wheel_joint">
+                <command_interface name="velocity">
+                    <param name="min">-10</param>
+                    <param name="max">10</param>
+                </command_interface>
+                <state_interface name="velocity"/>
+                <state_interface name="position"/>
+            </joint>
+            <joint name="right_wheel_joint">
+                <command_interface name="velocity">
+                    <param name="min">-10</param>
+                    <param name="max">10</param>
+                </command_interface>
+                <state_interface name="velocity"/>
+                <state_interface name="position"/>
+            </joint>
+        </ros2_control>
+    </xacro:if>
     <gazebo>
         <plugin name="gazebo_ros2_control" filename="libgazebo_ros2_control.so">
